File: GalaxySparkles.kicad_sch (KiCad schematic)
At the start: 111 parts, among them J1 Barrel_Jack, J2 STLINK-V3, J3 Debug Header, J4 USB_B, J5 FTDI (Expected), J6 FTDI (Reversed), J7 LEDS_MOS1, J8 LEDS_MOSI2, J9 LEDS_MOSI3, SW1 SW_SPDT, SW2 SW_Push, U1 STM32G0B1CEUx, U2 SN74LV1T34DBV, U3 SN74LV1T34DBV, U4 AP2112K-3.3, U5 SN74LV1T34DBV, U6 REF2030, Y2 32.768kHz

Commit message: v1.1 Updating to 24 LEDs & adding boot0 strap
Things done:
- Adjusted USB length a bit, now under 1mm difference, probably close
  enough
- Added a boot0 jumper point.  Don't need it per-se but it's a nice to
  have
- Moved from 18 LEDs to 24 LEDs on each chain

Signed-off-by: John 'Warthog9' Hawley <warthog9@eaglescrag.net>
Parts:
- added J10: boot0, Connector_PinHeader_2.54mm:PinHeader_1x02_P2.54mm_Vertical, symbol Connector_Generic:Conn_01x02
- added LED1-19, LED1-20, LED1-21, LED1-22, LED1-23, LED1-24, LED2-19, LED2-20, LED2-21, LED2-22, LED2-23, LED2-24, LED3-19, LED3-20, LED3-21, LED3-22, LED3-23, LED3-24: LTST-E133HEGBK, KiCad:LTSTE133HEGBK, symbol LTST-E133HEGBK:LTST-E133HEGBK
- added R10: 10K, Resistor_SMD:R_0805_2012Metric, symbol Device:R_US
- R8: LCSC C17414 -> C17408
Connections:
- net +3.3V: now also R10.2
- net GND: now also LED1-19.3 (VSS), LED1-20.3 (VSS), LED1-21.3 (VSS), LED1-22.3 (VSS), LED1-23.3 (VSS), LED1-24.3 (VSS), LED2-19.3 (VSS), LED2-20.3 (VSS), LED2-21.3 (VSS), LED2-22.3 (VSS), LED2-23.3 (VSS), LED2-24.3 (VSS), LED3-19.3 (VSS), LED3-20.3 (VSS), LED3-21.3 (VSS), LED3-22.3 (VSS), LED3-23.3 (VSS), LED3-24.3 (VSS)
- net SWCLK: now also J10.1 (Pin_1)
- net VBUS: now also LED1-19.1 (VDD), LED1-20.1 (VDD), LED1-21.1 (VDD), LED1-22.1 (VDD), LED1-23.1 (VDD), LED1-24.1 (VDD), LED2-19.1 (VDD), LED2-20.1 (VDD), LED2-21.1 (VDD), LED2-22.1 (VDD), LED2-23.1 (VDD), LED2-24.1 (VDD), LED3-19.1 (VDD), LED3-20.1 (VDD), LED3-21.1 (VDD), LED3-22.1 (VDD), LED3-23.1 (VDD), LED3-24.1 (VDD)
- net at LED2-18.4 (DOUT): now also LED2-19.2 (DIN)
- net at LED1-18.4 (DOUT): now also LED1-19.2 (DIN)
- net at LED3-18.4 (DOUT): now also LED3-19.2 (DIN)
- new net: LED3-19.4 (DOUT), LED3-20.2 (DIN)
- new net: LED3-20.4 (DOUT), LED3-21.2 (DIN)
- new net: LED2-21.4 (DOUT), LED2-22.2 (DIN)
- new net: LED2-22.4 (DOUT), LED2-23.2 (DIN)
- new net: J10.2 (Pin_2), R10.1
- new net: LED3-21.4 (DOUT), LED3-22.2 (DIN)
- new net: LED3-22.4 (DOUT), LED3-23.2 (DIN)
- new net: LED3-23.4 (DOUT), LED3-24.2 (DIN)
- new net: LED1-23.4 (DOUT), LED1-24.2 (DIN)
- new net: LED2-20.4 (DOUT), LED2-21.2 (DIN)
- new net: LED1-22.4 (DOUT), LED1-23.2 (DIN)
- new net: LED1-21.4 (DOUT), LED1-22.2 (DIN)
- new net: LED1-19.4 (DOUT), LED1-20.2 (DIN)
- new net: LED1-20.4 (DOUT), LED1-21.2 (DIN)
- new net: LED2-19.4 (DOUT), LED2-20.2 (DIN)
- new net: LED2-23.4 (DOUT), LED2-24.2 (DIN)
Other:
- note added: "Boot Mode boot0"
- moved on the sheet: C6, C7, LED2-1, LED2-10, LED2-11, LED2-12, LED2-13, LED2-14, LED2-15, LED2-16, LED2-17, LED2-18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
